File: schematic/blcd.kicad_sch (KiCad schematic)
At the start: 0 parts

Commit message: schematic in process
Other:
- note added: "Commercial Brushless DC motor driver"
- note added: "One IC is different on this one"
- note added: "Red and Black +24v & gnd Yellow is pwm signal 60% max duty cycle No feedback sensors Jumper by pot removed for PWM control Newer similar version with two caps and a push button"
